File: pcb/2D-EGGS.kicad_sch (KiCad schematic)
At the start: 55 parts, among them J1 ISP, J10 B10, J11 B8, J12 PWAN_CENTER_LED, J13 PWAN_E1P1, J14 PWAN_E1P2, J15 ENCODER1, J16 DPWR, J17 PWAN_E2P1, J18 PWAN_E2P2, J19 ENCODER2, J2 TT_LED, J20 B9, J21 B11, J22 PWAN_USB_B, J23 PWAN_USB_C, J24 LED1, J25 LED2, J26 APWR, J3 B1, J4 B6, J5 B3, J6 B4, J7 B5, J8 B2, J9 B7, P1 USB_C_DATA, P2 USB_C_POWER, Q10 2N7002, Q11 2N7002, Q12 2N7002, Q13 2N7002, Q3 2N7002, Q4 2N7002, Q5 2N7002, Q6 2N7002, Q7 2N7002, Q8 2N7002, Q9 2N7002, SW1 SW_Push, U1 AT90USB1286, Y1 16MHz

Commit message: fix unconnected pad on B11 MOSFET
Connections:
- net GND: now also Q10.2 (S)
Changed lines of the file:
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@@
   (junction (at 180.34 175.26) (diameter 0) (color 0 0 0 0)
   )
-  (junction (at 256.54 161.29) (diameter 0) (color 0 0 0 0)
-  )
   (junction (at 179.07 187.96) (diameter 0) (color 0 0 0 0)
   )
-  (junction (at 264.024 163.83) (diameter 0) (color 0 0 0 0)
-  )
   (junction (at 167.64 187.96) (diameter 0) (color 0 0 0 0)
   )
@@
     (stroke (width 0) (type default))
   )
+  (wire (pts (xy 231.14 163.83) (xy 264.16 163.83))
+    (stroke (width 0) (type default))
+  )
   (wire (pts (xy 172.72 62.23) (xy 172.72 74.93))
     (stroke (width 0) (type default))
@@
     (stroke (width 0) (type default))
   )
+  (wire (pts (xy 256.54 161.29) (xy 264.16 161.29))
+    (stroke (width 0) (type default))
+  )
   (wire (pts (xy 107.95 171.45) (xy 139.7 171.45))
     (stroke (width 0) (type default))
@@
     (stroke (width 0) (type default))
   )
-  (wire (pts (xy 264.024 161.29) (xy 256.54 161.29))
-    (stroke (width 0) (type default))
-  )
-  (wire (pts (xy 231.14 163.83) (xy 264.024 163.83))
-    (stroke (width 0) (type default))
-  )
   (wire (pts (xy 151.13 125.73) (xy 156.21 125.73))
     (stroke (width 0) (type default))
@@
     (stroke (width 0) (type default))
   )
-  (wire (pts (xy 256.54 161.29) (xy 256.404 161.29))
-    (stroke (width 0) (type default))
-  )
   (wire (pts (xy 217.17 146.05) (xy 231.14 146.05))
     (stroke (width 0) (type default))
@@
     (stroke (width 0) (type default))
   )
-  (wire (pts (xy 264.024 163.83) (xy 264.16 163.83))
-    (stroke (width 0) (type default))
-  )
   (wire (pts (xy 125.73 128.27) (xy 156.21 128.27))
     (stroke (width 0) (type default))
@@
     )
   )
-  (symbol (lib_id "power:+5V") (at 264.024 158.75 90) (unit 1)
+  (symbol (lib_id "power:+5V") (at 264.16 158.75 90) (unit 1)
     (in_bom yes) (on_board yes) (dnp no) (fields_autoplaced)
-    (property "Reference" "#PWR028" (at 267.834 158.75 0)
+    (property "Reference" "#PWR028" (at 267.97 158.75 0)
       (effects (font (size 1.27 1.27)) hide)
     )
-    (property "Value" "+5V" (at 260.214 158.115 90)
+    (property "Value" "+5V" (at 260.35 158.115 90)
       (effects (font (size 1.27 1.27)) (justify left))
     )
-    (property "Footprint" "" (at 264.024 158.75 0)
+    (property "Footprint" "" (at 264.16 158.75 0)
       (effects (font (size 1.27 1.27)) hide)
     )
-    (property "Datasheet" "" (at 264.024 158.75 0)
+    (property "Datasheet" "" (at 264.16 158.75 0)
       (effects (font (size 1.27 1.27)) hide)
     )
@@
     )
   )
-  (symbol (lib_id "power:GND") (at 246.244 161.29 270) (unit 1)
+  (symbol (lib_id "power:GND") (at 246.38 161.29 270) (unit 1)
     (in_bom yes) (on_board yes) (dnp no) (fields_autoplaced)
-    (property "Reference" "#PWR030" (at 239.894 161.29 0)
+    (property "Reference" "#PWR030" (at 240.03 161.29 0)
       (effects (font (size 1.27 1.27)) hide)
     )
-    (property "Value" "GND" (at 242.434 160.655 90)
+    (property "Value" "GND" (at 242.57 160.655 90)
       (effects (font (size 1.27 1.27)) (justify right))
     )
-    (property "Footprint" "" (at 246.244 161.29 0)
+    (property "Footprint" "" (at 246.38 161.29 0)
       (effects (font (size 1.27 1.27)) hide)
     )
-    (property "Datasheet" "" (at 246.244 161.29 0)
+    (property "Datasheet" "" (at 246.38 161.29 0)
       (effects (font (size 1.27 1.27)) hide)
     )
@@
     )
   )
-  (symbol (lib_id "power:GND") (at 264.024 156.21 270) (unit 1)
+  (symbol (lib_id "power:GND") (at 264.16 156.21 270) (unit 1)
     (in_bom yes) (on_board yes) (dnp no) (fields_autoplaced)
-    (property "Reference" "#PWR029" (at 257.674 156.21 0)
+    (property "Reference" "#PWR029" (at 257.81 156.21 0)
       (effects (font (size 1.27 1.27)) hide)
     )
-    (property "Value" "GND" (at 260.214 155.575 90)
+    (property "Value" "GND" (at 260.35 155.575 90)
       (effects (font (size 1.27 1.27)) (justify right))
     )
-    (property "Footprint" "" (at 264.024 156.21 0)
+    (property "Footprint" "" (at 264.16 156.21 0)
       (effects (font (size 1.27 1.27)) hide)
     )
-    (property "Datasheet" "" (at 264.024 156.21 0)
+    (property "Datasheet" "" (at 264.16 156.21 0)
       (effects (font (size 1.27 1.27)) hide)
     )
@@
     )
   )
-  (symbol (lib_id "Connector:Conn_01x04_Pin") (at 269.104 161.29 180) (unit 1)
+  (symbol (lib_id "Connector:Conn_01x04_Pin") (at 269.24 161.29 180) (unit 1)
     (in_bom yes) (on_board yes) (dnp no)
-    (property "Reference" "J10" (at 271.644 161.29 0)
+    (property "Reference" "J10" (at 271.78 161.29 0)
       (effects (font (size 1.27 1.27)))
     )
-    (property "Value" "B10" (at 271.78 158.75 0)
+    (property "Value" "B10" (at 271.916 158.75 0)
       (effects (font (size 1.27 1.27)))
     )
-    (property "Footprint" "Connector_JST:JST_XH_B4B-XH-A_1x04_P2.50mm_Vertical" (at 269.104 161.29 0)
+    (property "Footprint" "Connector_JST:JST_XH_B4B-XH-A_1x04_P2.50mm_Vertical" (at 269.24 161.29 0)
       (effects (font (size 1.27 1.27)) hide)
     )
-    (property "Datasheet" "~" (at 269.104 161.29 0)
+    (property "Datasheet" "~" (at 269.24 161.29 0)
       (effects (font (size 1.27 1.27)) hide)
     )
