File: remote-board/remote-board.kicad_pcb (KiCad board)
At the start: 2 copper layers, 52 x 25 mm, 5 parts, among them J1 USB1JST, J2 USB2JST, J3 USB_B, J4 USB_B

Commit message: [remote-board] fix reversed JST wiring
Parts:
- moved J1 35.0 mm to (129.9, 103.6)
- moved J2 35.0 mm to (154.3, 103.6)
- moved J3 35.0 mm to (132.6, 97.8)
- moved J4 35.0 mm to (156.7, 97.8)
- moved G*** 35.0 mm to (145.8, 104.5)
Connections:
- J1 pad 1: GND -> Net-(J1-Pin_1)
- J1 pad 2: /USB1_D+ -> /USB1_D-
- J1 pad 3: /USB1_D- -> /USB1_D+
- J1 pad 4: Net-(J1-Pin_4) -> GND
- J2 pad 1: GND -> Net-(J2-Pin_1)
- J2 pad 2: /USB2_D+ -> /USB2_D-
- J2 pad 3: /USB2_D- -> /USB2_D+
- J2 pad 4: Net-(J2-Pin_4) -> GND
- J3 pad 1: Net-(J1-Pin_4) -> Net-(J1-Pin_1)
- J4 pad 1: Net-(J2-Pin_4) -> Net-(J2-Pin_1)
Routing:
- net Net-(J2-Pin_4): track 9.36 -> 0.00 mm
- net Net-(J1-Pin_4): track 9.09 -> 0.00 mm
- net Net-(J1-Pin_1): track 0.00 -> 6.97 mm
- net Net-(J2-Pin_1): track 0.00 -> 6.85 mm
- net /USB2_D-: track 8.04 -> 6.85 mm
- net /USB1_D-: track 9.06 -> 7.87 mm
