File: remote-board/remote-board.kicad_sch (KiCad schematic)
At the start: 4 parts, among them J1 USB1JST, J2 USB2JST, J3 USB_B, J4 USB_B

Commit message: [remote-board] fix reversed JST wiring
Connections:
- net GND: now also J1.4 (Pin_4), J2.4 (Pin_4); no longer J1.1 (Pin_1), J2.1 (Pin_1)
- net USB1_D+: now also J1.3 (Pin_3); no longer J1.2 (Pin_2)
- net USB1_D-: now also J1.2 (Pin_2); no longer J1.3 (Pin_3)
- net USB2_D+: now also J2.3 (Pin_3); no longer J2.2 (Pin_2)
- net USB2_D-: now also J2.2 (Pin_2); no longer J2.3 (Pin_3)
- net at J4.1 (VBUS): now also J2.1 (Pin_1); no longer J2.4 (Pin_4)
- net at J3.1 (VBUS): now also J1.1 (Pin_1); no longer J1.4 (Pin_4)
Other:
- moved on the sheet: J1, J2
